File: kicad/1550Z124.kicad_pcb (KiCad board)
At the start: 2 copper layers, 213.3 x 96 mm, 153 parts, among them J1 Conn_02x07_Odd_Even, J2 Conn_01x02, K1 Fujitsu_FTR-K1C, K10 Fujitsu_FTR-K1C, K11 Fujitsu_FTR-K1C, K12 Fujitsu_FTR-K1C, K13 Fujitsu_FTR-K1C, K14 Fujitsu_FTR-K1C, K15 Fujitsu_FTR-K1C, K16 Fujitsu_FTR-K1C, K17 Fujitsu_FTR-K1C, K18 Fujitsu_FTR-K1C, K2 Fujitsu_FTR-K1C, K3 Fujitsu_FTR-K1C, K4 Fujitsu_FTR-K1C, K5 Fujitsu_FTR-K1C, K6 Fujitsu_FTR-K1C, K7 Fujitsu_FTR-K1C, K8 Fujitsu_FTR-K1C, K9 Fujitsu_FTR-K1C, Q1 BC817, Q10 BC817, Q11 BC817, Q12 BC817, Q2 BC817, Q3 BC817, Q4 BC817, Q5 BC817, Q6 BC817, Q7 BC817, Q8 BC817, Q9 BC817

Commit message: vias, lots of vias
Routing:
- net GND: track 203.0 -> 194.5 mm, vias 2791 -> 2795
Changed lines of the file:
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@@
     (thickness 1.6)
     (drawings 166)
-    (tracks 3566)
+    (tracks 3568)
     (zones 0)
     (modules 153)
@@
   (segment (start 222.09 106.8) (end 222.09 114.3) (width 2.54) (layer F.Cu) (net 1))
   (segment (start 257.015 114.3) (end 257.015 106.8) (width 2.54) (layer F.Cu) (net 1))
-  (segment (start 291.94 106.8) (end 293.5224 113.1062) (width 2.54) (layer F.Cu) (net 1))
   (segment (start 130.92 139.81) (end 131.335 139.81) (width 2.54) (layer F.Cu) (net 1))
   (segment (start 130.81 121.92) (end 130.92 121.81) (width 2.54) (layer F.Cu) (net 1))
@@
   (segment (start 291.94 114.3) (end 291.94 114.3) (width 2.54) (layer F.Cu) (net 1))
   (via (at 291.94 114.3) (size 0.8) (drill 0.4) (layers F.Cu B.Cu) (net 1))
-  (segment (start 293.5224 113.1062) (end 291.94 114.3) (width 2.54) (layer F.Cu) (net 1))
   (via (at 293.5224 113.1062) (size 0.8) (drill 0.4) (layers F.Cu B.Cu) (net 1))
   (via (at 294.7924 116.9162) (size 0.8) (drill 0.4) (layers F.Cu B.Cu) (net 1))
@@
   (via (at 266.8524 161.3662) (size 0.8) (drill 0.4) (layers F.Cu B.Cu) (net 1))
   (via (at 268.1224 166.4462) (size 0.8) (drill 0.4) (layers F.Cu B.Cu) (net 1))
+  (via (at 292.2524 109.2962) (size 0.8) (drill 0.4) (layers F.Cu B.Cu) (net 1))
+  (via (at 293.5224 110.5662) (size 0.8) (drill 0.4) (layers F.Cu B.Cu) (net 1))
+  (via (at 290.9824 110.5662) (size 0.8) (drill 0.4) (layers F.Cu B.Cu) (net 1))
+  (via (at 292.2524 111.8362) (size 0.8) (drill 0.4) (layers F.Cu B.Cu) (net 1))
   (segment (start 107.87 125.73) (end 107.95 125.65) (width 2.54) (layer B.Cu) (net 2))
   (segment (start 107.95 125.65) (end 115.45 125.65) (width 2.54) (layer F.Cu) (net 2))
