File: kicad/antenna_switch/antenna_switch.kicad_pcb (KiCad board)
At the start: 2 copper layers, 213.3 x 96 mm, 154 parts, among them J1 Conn_02x07_Odd_Even, J2 Conn_01x02, K1 Fujitsu_FTR-K1C, K10 Fujitsu_FTR-K1C, K11 Fujitsu_FTR-K1C, K12 Fujitsu_FTR-K1C, K13 Fujitsu_FTR-K1C, K14 Fujitsu_FTR-K1C, K15 Fujitsu_FTR-K1C, K16 Fujitsu_FTR-K1C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

Commit message: Updated README
Other:
- net class Default removed
