File: kicad/antenna_switch_comms/antenna_switch_comms.kicad_pcb (KiCad board)
At the start: 2 copper layers, 70 x 96 mm, 44 parts, among them J1 AVR-ISP-6, J2 Conn_02x07_Odd_Even, J3 Conn_01x02, J4 Conn_01x02, SW1 SW_Push, U1 ATmega328P-AU, U2 MAX13487, U3 MC7805BDTRKG, Y1 16M

Commit message: Updated README
Other:
- net class Default removed
