File: kicad/esp32_comms/esp32.kicad_sch (KiCad schematic)
At the start: 7 parts, among them J2 Conn_02x07_Odd_Even, SW1 SW_Push

Commit message: ESP32 Interface Module HW
Parts:
- added J201: Conn_02x03, Connector_PinHeader_2.54mm:PinHeader_2x03_P2.54mm_Vertical, symbol PCM_4ms_Connector:Conn_02x03
- added R201, R202: 10k, Resistor_SMD:R_0805_2012Metric_Pad1.20x1.40mm_HandSolder, symbol Device:R_Small
- C201: LCSC Part # (none) -> C12891
- C202: footprint Capacitor_SMD:C_0805_2012Metric_Pad1.18x1.45mm_HandSolder -> Capacitor_SMD:C_0805_2012Metric_Pad1.15x1.40mm_HandSolder; LCSC Part # (none) -> C49678
- D10: LCSC Part # (none) -> C2297
- R9: LCSC Part # (none) -> C17710
Connections:
- net +5V: now also U201.15 (VIN); no longer U201.1 (VIN)
- net A1R1: now also U201.13 (GPIO13); no longer U201.8 (GPIO25)
- net A2R1: now also U201.12 (GPIO12); no longer U201.7 (GPIO26)
- net A3R1: now also U201.11 (GPIO14); no longer U201.6 (GPIO27)
- net A4R1: now also U201.10 (GPIO27); no longer U201.5 (GPIO14)
- net A5R1: now also U201.9 (GPIO26); no longer U201.4 (GPIO12)
- net A6R1: now also U201.8 (GPIO25); no longer U201.3 (GPIO13)
- net GND: now also U201.14 (GND), J201.2 (+12V); no longer U201.2 (GND)
- net at SW1.2: now also U201.1 (EN); no longer U201.15 (EN)
- net at D10.2 (A): now also U201.6 (GPIO32); no longer U201.10 (GPIO32)
- net +3V3: now reaches U201.16 (3.3v)
- net +3V3: now also J201.1 (+12V), R201.1, R202.1
- net GPIO15: now reaches U201.18 (GPIO15)
- net GPIO15: now also J201.5 (GND)
- net SDA: now reaches U201.19 (GPIO2)
- net SDA: now also J201.3 (GND), R202.2
- net SCL: now reaches U201.20 (GPIO4)
- net SCL: now also J201.4 (GND), R201.2
- new net GPIO33: J201.6 (GND), U201.7 (GPIO33)
Other:
- note added: "Relay Module Connector"
- note added: "Simple AddOn Connector"
- company: (none) -> SQ9NJE Quirky Solutions
- title: (none) -> ESP32
- moved on the sheet: C201, C202, D10, J2, R9, SW1
