File: kicad/esp32_comms/esp32_comms.kicad_pcb (KiCad board)
At the start: 2 copper layers, 70 x 96 mm, 38 parts, among them J2 Conn_02x07_Odd_Even, J3 Conn_01x02, J4 Conn_01x02, SW1 SW_Push, U2 MAX13487, U3 LM7805_TO220

Commit message: ESP32 Interface Module HW
Parts:
- added FID101: Fiducial, Fiducial:Fiducial_1mm_Mask2mm, F.Cu at (105.0, 105.0)
- added FID102: Fiducial, Fiducial:Fiducial_1mm_Mask2mm, F.Cu at (105.0, 191.0)
- added FID103: Fiducial, Fiducial:Fiducial_1mm_Mask2mm, F.Cu at (165.0, 105.0)
- added J201: Conn_02x03, Connector_PinHeader_2.54mm:PinHeader_2x03_P2.54mm_Vertical, F.Cu at (157.5, 179.8)
- added R201: 10k, Resistor_SMD:R_0805_2012Metric_Pad1.20x1.40mm_HandSolder, F.Cu at (141.5, 184.8)
- added R202: 10k, Resistor_SMD:R_0805_2012Metric_Pad1.20x1.40mm_HandSolder, F.Cu at (145.0, 184.8)
- D2, D4, D5, D6: value TESDU24V -> TSDU24V
- H101, H102, H103, H104: renamed from REF**; value MountingHole_3.2mm_M3_ISO7380_Pad -> MountingHole_Pad
- JP1, JP2: footprint Connector_PinHeader_2.54mm:PinHeader_1x02_P2.54mm_Vertical -> Jumper:SolderJumper-2_P1.3mm_Bridged_RoundedPad1.0x1.5mm
- moved C202 33.9 mm to (125.2, 184.8), turned to 90 degrees
- moved C201 33.4 mm to (119.5, 184.7), turned to 90 degrees
- moved SW1 28.4 mm to (112.8, 150.2)
- moved Ref** 4.66 mm to (110.0, 162.8), turned to -90 degrees
- moved JP1 0.95 mm to (126.5, 122.3)
- moved JP2 0.91 mm to (123.8, 122.3), turned to 90 degrees
Connections:
- U201 pad 1: +5V -> Net-(U201-EN)
- U201 pad 10: Net-(D10-A) -> A4R1
- U201 pad 11: unconnected-(U201-GPIO35-Pad11) -> A3R1
- U201 pad 12: unconnected-(U201-GPIO34-Pad12) -> A2R1
- U201 pad 13: unconnected-(U201-GPIO39-Pad13) -> A1R1
- U201 pad 14: unconnected-(U201-GPIO36-Pad14) -> GND
- U201 pad 15: Net-(U201-EN) -> +5V
- U201 pad 16: unconnected-(U201-3.3v-Pad16) -> +3V3
- U201 pad 18: unconnected-(U201-GPIO15-Pad18) -> /ESP32/GPIO15
- U201 pad 19: unconnected-(U201-GPIO2-Pad19) -> /ESP32/SDA
- U201 pad 2: GND -> unconnected-(U201-GPIO36-Pad2)
- U201 pad 20: unconnected-(U201-GPIO4-Pad20) -> /ESP32/SCL
- U201 pad 3: A6R1 -> unconnected-(U201-GPIO39-Pad3)
- U201 pad 4: A5R1 -> unconnected-(U201-GPIO34-Pad4)
- U201 pad 5: A4R1 -> unconnected-(U201-GPIO35-Pad5)
- U201 pad 6: A3R1 -> Net-(D10-A)
- U201 pad 7: A2R1 -> /ESP32/GPIO33
- U201 pad 8: A1R1 -> A6R1
- U201 pad 9: unconnected-(U201-GPIO33-Pad9) -> A5R1
Routing:
- net /ESP32/GPIO33: track 0.00 -> 44.8 mm
- net +5V: track 95.9 -> 138.0 mm, vias 0 -> 1
- net /ESP32/SCL: track 0.00 -> 23.3 mm
- net /ESP32/SDA: track 0.00 -> 19.3 mm
- net +3V3: track 0.00 -> 18.6 mm
- net /ESP32/GPIO15: track 0.00 -> 15.8 mm
- net Net-(D10-A): track 49.1 -> 39.0 mm
- net Net-(U201-EN): track 13.1 -> 5.89 mm
- net GND: track 0.00 -> 5.99 mm, vias 396 -> 386
- net RS485_A: track 24.5 -> 19.9 mm, vias 0 -> 2
- net RS485_B: track 24.5 -> 20.1 mm, vias 0 -> 2
- net A4R1: track 39.8 -> 44.0 mm
- net A3R1: track 39.8 -> 44.0 mm
- net A2R1: track 39.8 -> 44.0 mm
- net A5R1: track 39.8 -> 44.0 mm
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Other:
- board text added: "3V3"
- board text added: "A"
- board text added: "B"
- board text added: "IO15"
- board text added: "IO33"
- board text added: "RS485"
- board text added: "SAO"
- board text added: "SCL"
- board text added: "SDA"
