File: kicad/esp32_comms/esp32_comms.kicad_sch (KiCad schematic)
At the start: 0 parts

Commit message: ESP32 Interface Module HW
Parts:
- added FID101, FID102, FID103: Fiducial, Fiducial:Fiducial_1mm_Mask2mm, symbol Mechanical:Fiducial
- added H101, H102, H103, H104: MountingHole_Pad, MountingHole:MountingHole_3.2mm_M3_ISO7380_Pad, symbol Mechanical:MountingHole_Pad
Connections:
- net GND: now also H101.1, H102.1, H103.1, H104.1
Other:
- title: 6x2 Matrix Antenna Switch - Communication Module -> 6x2 Matrix Antenna Switch - Interface Module
