File: kicad/esp32_comms/psu.kicad_sch (KiCad schematic)
At the start: 11 parts, among them J3 Conn_01x02, U3 LM7805_TO220

Commit message: ESP32 Interface Module HW
Parts:
- C11, C9: LCSC Part # (none) -> C49678
- D2: value TESDU24V -> TSDU24V; LCSC Part # (none) -> C2836324
- D3: LCSC Part # (none) -> C2480
- D8: LCSC Part # (none) -> C2297
- F1: LCSC Part # (none) -> C269104
- R7: LCSC Part # (none) -> C17520
Other:
- company: (none) -> SQ9NJE Quirky Solutions
- title: (none) -> Power Supply
- moved on the sheet: C10, C11, C8, C9, D2, D3, D8, F1, J3, R7, U3
