File: kicad/esp32_comms/rs485.kicad_sch (KiCad schematic)
At the start: 15 parts, among them J4 Conn_01x02, U2 MAX13487

Commit message: ESP32 Interface Module HW
Parts:
- C7: LCSC Part # (none) -> C49678
- D4, D5, D6: value TESDU24V -> TSDU24V; LCSC Part # (none) -> C2836324
- D7, D9: LCSC Part # (none) -> C2297
- JP1, JP2: footprint Connector_PinHeader_2.54mm:PinHeader_1x02_P2.54mm_Vertical -> Jumper:SolderJumper-2_P1.3mm_Bridged_RoundedPad1.0x1.5mm; now left out of the parts list
- R3, R8: LCSC Part # (none) -> C17520
- R4, R6: LCSC Part # (none) -> C17513
- R5: LCSC Part # (none) -> C17437
- U2: LCSC Part # (none) -> C18347
Other:
- company: (none) -> SQ9NJE Quirky Solutions
- title: (none) -> RS485 Interface
- moved on the sheet: C7, D4, D5, D6, D7, D9, J4, JP1, JP2, R3, R4, R5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
